File: m2_simcom_7100.sch (KiCad schematic (older format))
At the start: 4 parts, among them J1 M.2_Key_B

Commit message: add SIM7100 schematic symbol
Parts:
- added U?: SIM7100, symbol SIM7100
Other:
- moved on the sheet: J1

Commit message: Save progress just before replacing pins 10, 23, 25, 26, 44, 46, and 48 with UART pins due to it being Port Configuration 3 / State 7 (no GNSS)
Pins 10 ~LED1 and 25 DPR (DPR unavailable anyway) being the most practical alternate functions
Pin 26 was ~W_Disable2 but it was unused anyway, and even if it were it would meant for GNSS anyway (~W_Disable1 takes care of both here)
Parts:
- removed ANT1, ANT2, ANT4: Conn_Coaxial, m2_key_b_3042:MHF4_20449-001E, symbol Conn_Coaxial
- added AE?: Main_Antenna, symbol Antenna_Shield
- added AE?: GNSS_Antenna, symbol Antenna_Shield
- added AE?: Div_Antenna, symbol Antenna_Shield
- added C? (x4): NC, symbol C
- added C? (x2): 100uF, symbol CP1
- added C? (x2): 100uF, symbol C
- added C?: 1uF, symbol C
- added C?: 33pF, symbol C
- added C? (x2): 100nF, symbol C
- added D?: D_TVS, symbol D_TVS
- added J? (x2): TEST_1P, symbol TEST_1P
- added L? (x2): NC, symbol L
- added Q? (x2): Q_NPN_BCE, symbol Q_NPN_BCE
- added R? (x2): 0, symbol R
- added R? (x2): 10k, symbol R
- added R? (x2): 47k, symbol R
- added R? (x3): 51, symbol R
Connections:
- net labels added: DPR/GPIO_12, GPIO_10/~W_Disable2, GPIO_2/GNSS_IRQ, GPIO_3/SYSCLK, GPIO_4/TX_BLANKING, HSIC_Data, HSIC_Strobe, PCM_CLK, PCM_IN, PCM_OUT, PCM_SYNC, Status, UART_CTS, UART_DCD, UART_DTR, UART_RI/~WoWWAN, UART_RTS, UART_RX, UART_TX, USB3.0-Rx+, USB3.0-Rx-, USB3.0-Tx+, USB3.0-Tx-, USB_VBUS, VBUS, ~LED1
- net labels removed: AUX, DEVSLP, GPIO_0, GPIO_1, GPIO_10, GPIO_11, GPIO_12, GPIO_2, GPIO_3, GPIO_4, GPIO_5, GPIO_6, GPIO_7, GPIO_8, GPIO_9/DAS/~DSS, GPS, MAIN, PERn0/SATA-B+, PERn1/USB3.0-Rx-/SSIC-RxN, PERp0/SATA-B-, PERp1/USB3.0-Rx+/SSIC-RxP, PETn0/SATA-A-, PETn1/USB3.0-Tx-/SSIC-TxN, PETp0/SATA-A+, PETp1/USB3.0-Tx+/SSIC-TxP, REFCLKN, REFCLKP, ~CLKREQ, ~PERST, ~PEWake
- wire segments 77 -> 241
- no-connect marks 54 -> 59
Other:
- note added: "5V Regulator!!!"
- note added: "Can be swapped\naround in layout"
- note added: "ESD protection near card\nCaps on VDD of SIM"
- note added: "Find AT Command to set TX Power\nNot TXPWR Parameter (read-only)!\nModule does not have DPR"
- note added: "May Use Boost\nEN Pin Instead\nNeeds 3.3V Tolerance!"
- note added: "Not Provided"
- note added: "Port Configuration 3 / State 7\n (Audio + HSIC, no GNSS)"
- note added: "Traced by 90Ohm+/-10%\nDifferential Impedance!"
- note added: "Used Table 30"
- note removed: "(Used Table 48)\nCHECK TABLE 29/30!!!"
- note removed: "???"
- moved on the sheet: J1, U?

Commit message: Remove GNSS antenna circuit and place notes regarding external circuit
Add power sheet for the boost converter for Vbat (3.8V) and Vbus (tie to Vbat)
Parts:
- removed AE?: GNSS_Antenna, symbol Antenna_Shield
- removed C?: 33pF, symbol C
- removed L? (x2): NC, symbol L
- removed Q?: Q_NPN_BCE, symbol Q_NPN_BCE
- removed R? (x2): 10k, symbol R
- added D2: ESD9L5.0ST5G, symbol D_Zener_Small_ALT
- gave numbers to parts that had none: 25
Connections:
- net labels added: Netlight/LED1, VBAT
- net labels removed: DPR/GPIO_12, GPIO_10/~W_Disable2, GPIO_2/GNSS_IRQ, GPIO_3/SYSCLK, GPIO_4/TX_BLANKING, VBUS, ~LED1
- wire segments 241 -> 173
- no-connect marks 59 -> 60
Other:
- note added: "Add same TVS Diode to\nUSB_D± on Main Board"
- note added: "CLK xtrnl NC Cap to GND"
- note added: "Can transmit PCM\ndata over USB!"
- note added: "ESD protection near card\n100nF on VDD of SIM"
- note added: "Implemented by\ncard holder"
- note added: "Module Table 30 &\nmPCIe 3.6 note 2\nsays this is fine"
- note added: "Pull Up RI/WoWWAN on\nthe Host Side to 1.8V"
- note added: "Suggests WM8960 CODEC\nwith SIM7100 connected\nover I2C?!"
- note added: "~W_DISABLE1\nExternal Circuit\nFigure 5"
- note removed: ""HSIC supported on WWAN configuration 3""
- note removed: "5V Regulator!!!"
- note removed: "ESD protection near card\nCaps on VDD of SIM"
- note removed: "Huawei MU736 is an example of 3G M.2 card which supports SSIC\nThe i.MX 8M does not explicity state SSIC support"
- note removed: "Unfortunately, it seems most WWAN modules don't explicitly support SSIC\nThis will need to be looked into:\n"SSIC brings 80% power savings using a MIPI\n M-PHY and SSIC, as compared to a USB 3.0 PHY""
- moved on the sheet: AE1, AE2, C1, C10, C11, C2, C3, C4, C5, C6, C7, C8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

Commit message: Add MIC29302 LDO, VBAT will be used instead of 3.3V in order to reduce power consumption.
When testing this will require a ~3.8V supply at the M.2 connector!
Parts:
- added R3: 10k, symbol R
- C5: renamed from C4; value 100nF -> DNP
- D1: value D_TVS -> DNP
- Q1: value Q_NPN_BCE -> DNP
- R1, R2: value 47k -> DNP
- renumbered C3 to C2, C2 to C3, C5 to C4, J2 to J1, J3 to J2, J1 to J3, R3 to R4, R4 to R5, R5 to R6, R6 to R7, R7 to R8
Connections:
- net USB_VBUS is gone; now on net VBAT_REG: D2.1 (K), U1.11 (USB_VBUS)
- net GND: now also R3.2
- net ~Full_Card_Power_Off: no longer R1.1
- net at C5.1, D1.2 (A2), Q1.2 (C)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: now also R3.1
- net VBAT_REG: now reaches C11.1, C8.1, C9.1, U1.38 (VBAT), U1.39 (VBAT)
- net VBAT_REG: now also C1.1, C2.1, C4.1, U1.62 (VBAT), U1.63 (VBAT)
- net +3V3 renamed VBAT
- no-connect marks 60 -> 61
Other:
- note added: ""Alternatively, and primarily for Tablet\nplatforms, the 3.3 V regulated power rail can\nbe replaced with a direct VBAT connection."\n- M.2 Spec Table 41"
- note added: "Get Doc [26]"
- note added: "SIM7100A User Manual\nTable 9 note"
- note added: "Suggests NAU8810 CODEC\nwith SIM7100 connected\nover I2C?!"
- note added: "~Reset\nFigure 14 module\nFigure 4 xtrnl ckt"
- note removed: "May Use Boost\nEN Pin Instead\nNeeds 3.3V Tolerance!"
- note removed: "Suggests WM8960 CODEC\nwith SIM7100 connected\nover I2C?!"
- moved on the sheet: C1, C2, C4, Q1, R1, R2, R4

Commit message: Selected which bulk capacitors will be used throughout the design, allowing for a small profile with high capacitance and fast transient response time (low ESR/ESL); also created the respective footprint
Put in a few notes regarding discrepancies between what the SIM7100 documentation suggests for cap values and what the MIC29302 datasheet says. I chose to go wivalues closer to what SIM7100 suggests but with a lower output cap value due to what photos of the mPCIe module shows. Namely, use of a few TMCUB0J107MTRF 100uF caps throughout the design, using this same cap near the regulator in place of an expensive 330uF one (as suggested in figure 9).
Parts:
- removed C2, C9: 100uF, symbol C
- added C1, C9: 100uF, m2_simcom_7100:CP_Tantalum_Case-B_EIA-3528-21_Reflow, symbol CP1
- added D1: MMSZ5231BT1G, symbol D_Zener_Small_ALT
- added FB1: Ferrite, symbol Ferrite_Bead_Small
- ANT1: renamed from AE2; footprint (none) -> m2_simcom_7100:MHF4_20449-001E
- ANT4: renamed from AE1; footprint (none) -> m2_simcom7100:MHF4_20449-001E
- C11: renamed from C8; footprint (none) -> m2_simcom_7100:CP_Tantalum_Case-B_EIA-3528-21_Reflow
- C3: renamed from C1; value 100uF -> NC; footprint (none) -> m2_simcom_7100:CP_Tantalum_Case-B_EIA-3528-21_Reflow
- C4: renamed from C5; value DNP -> NC
- D2: renamed from D1; value DNP -> NC
- Q1, R1, R2: value DNP -> NC
- renumbered C3 to C2, C4 to C5, C11 to C8, D2 to D3, R5 to R4, R6 to R5, R4 to R6
Connections:
- net GND: now also C1.2, C9.2, D1.2 (A)
- net VBAT_REG: now also C9.1, D1.1 (K), FB1.2; no longer C3.1, C5.1, U1.62 (VBAT), U1.63 (VBAT)
- new net: C1.1, C3.1, C5.1, FB1.1, U1.62 (VBAT), U1.63 (VBAT)
Other:
- note added: "Figure 8"
- note added: "Suggests NAU8810 CODEC\nwith SIM7100 connected\nto I2C?!"
- note added: "~W_DISABLE1\nExternal Circuit\nmPCIe Figure 5"
- note removed: "Suggests NAU8810 CODEC\nwith SIM7100 connected\nover I2C?!"
- note removed: "~W_DISABLE1\nExternal Circuit\nFigure 5"
- moved on the sheet: C11, C3, C8

Commit message: Assign all footprints and generate netlist
Parts:
- removed D2: NC, symbol D_TVS
- added D2: NC, m2_simcom_7100:D_0402, symbol D_TVS_ALT
- C10, C5, C6, C7, C8: footprint (none) -> Capacitors_SMD:C_0603
- C2: renamed from C4; footprint (none) -> Capacitors_SMD:C_0603
- C3: renamed from C2; footprint (none) -> Capacitors_SMD:C_0603
- D1: footprint (none) -> m2_simcom_7100:D_SOD-123
- D3: footprint (none) -> m2_simcom_7100:D_SOD-923
- FB1: footprint (none) -> Inductors_SMD:L_0603
- Q1: footprint (none) -> TO_SOT_Packages_SMD:SOT-23
- R1, R2, R8: footprint (none) -> Resistors_SMD:R_0603
- R3: renamed from R4; footprint (none) -> Resistors_SMD:R_0603
- R4: renamed from R5; footprint (none) -> Resistors_SMD:R_0603
- R5: renamed from R6; footprint (none) -> Resistors_SMD:R_0603
- R6: renamed from R7; footprint (none) -> Resistors_SMD:R_0603
- R7: renamed from R3; footprint (none) -> Resistors_SMD:R_0603
- TP1: renamed from J1; footprint (none) -> Measurement_Points:Measurement_Point_Round-SMD-Pad_Small
- TP2: renamed from J2; footprint (none) -> Measurement_Points:Measurement_Point_Round-SMD-Pad_Small
- U1: footprint (none) -> m2_simcom_7100:SIMCom_7100
- renumbered ANT4 to ANT1, ANT1 to ANT2, C3 to C4, J3 to J1
Connections:
- net GND: now also D2.2 (A2)
- net at C2.1, Q1.2 (C), R7.1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: now also D2.1 (A1)
Other:
- moved on the sheet: C2, D1, FB1, Q1, R1, R2, R7

Commit message: Fix footprint associations in netlist which are pointing to the wrong library name
Parts:
- ANT5: renamed from ANT1; footprint m2_simcom7100:MHF4_20449-001E -> m2_simcom_7100:MHF4_20449-001E
- J1: footprint m2_key_b_3042:M.2_Key_B_Gold_Fingers -> m2_simcom_7100:M.2_Key_B_Gold_Fingers
Changed lines of the file:
@@
 F 0 "J1" H 9100 4900 50  0000 C CNN
 F 1 "M.2_Key_B" H 9100 1000 50  0000 C CNN
-F 2 "m2_key_b_3042:M.2_Key_B_Gold_Fingers" H 9050 3000 50  0001 C CNN
+F 2 "m2_simcom_7100:M.2_Key_B_Gold_Fingers" H 9050 3000 50  0001 C CNN
 F 3 "" H 9050 3000 50  0001 C CNN
 	1    9050 3000
@@
 $EndComp
 $Comp
-L Antenna_Shield ANT1
+L Antenna_Shield ANT5
 U 1 1 5AB020C9
 P 3600 800
-F 0 "ANT1" H 3525 975 50  0000 R CNN
+F 0 "ANT5" H 3525 975 50  0000 R CNN
 F 1 "Main_Antenna" H 3525 900 50  0000 R CNN
-F 2 "m2_simcom7100:MHF4_20449-001E" H 3600 900 50  0001 C CNN
+F 2 "m2_simcom_7100:MHF4_20449-001E" H 3600 900 50  0001 C CNN
 F 3 "https://www.mouser.com/ds/2/398/RECE.20449.001E.01-27117.pdf" H 3600 900 50  0001 C CNN
 	1    3600 800

Commit message: Swap Main and Div antenna positions
Parts:
- renumbered ANT5 to ANT2, ANT2 to ANT5
Changed lines of the file:
@@
 $EndComp
 $Comp
-L Antenna_Shield ANT5
+L Antenna_Shield ANT2
 U 1 1 5AB020C9
 P 3600 800
-F 0 "ANT5" H 3525 975 50  0000 R CNN
+F 0 "ANT2" H 3525 975 50  0000 R CNN
 F 1 "Main_Antenna" H 3525 900 50  0000 R CNN
 F 2 "m2_simcom_7100:MHF4_20449-001E" H 3600 900 50  0001 C CNN
@@
 $EndComp
 $Comp
-L Antenna_Shield ANT2
+L Antenna_Shield ANT5
 U 1 1 5AB09ED5
 P 6650 1550
-F 0 "ANT2" H 6600 1650 50  0000 R CNN
+F 0 "ANT5" H 6600 1650 50  0000 R CNN
 F 1 "Div_Antenna" H 6600 1550 50  0000 R CNN
 F 2 "m2_simcom_7100:MHF4_20449-001E" H 6650 1650 50  0001 C CNN
