File: power.sch (KiCad schematic (older format))
At the start: 10 parts, among them U2 RT9059

Commit message: Add 74AUP1G04 schmitt-triggered inverter to SIM_DET based on the fact that most WWAN M.2 modules expect this to be an active HIGH input
Parts:
- renumbered C12 to C13, C13 to C14, C14 to C15, C15 to C16, C16 to C17, R9 to R10, R10 to R11, R11 to R12, U2 to U3
Changed lines of the file:
@@
 encoding utf-8
 Sheet 2 2
-Title ""
-Date ""
-Rev ""
-Comp ""
-Comment1 ""
-Comment2 ""
+Title "Power"
+Date "2018-03-20"
+Rev "0.5.0"
+Comp "Purism SPC"
+Comment1 "Copyright 2018"
+Comment2 "GNU GPLv3"
 Comment3 ""
 Comment4 ""
 $EndDescr
 $Comp
-L GND #PWR021
+L GND #PWR025
 U 1 1 5AB193E7
 P 5950 4800
-F 0 "#PWR021" H 5950 4550 50  0001 C CNN
+F 0 "#PWR025" H 5950 4550 50  0001 C CNN
 F 1 "GND" H 5950 4650 50  0000 C CNN
 F 2 "" H 5950 4800 50  0001 C CNN
@@
 $EndComp
 $Comp
-L CP1 C12
+L CP1 C13
 U 1 1 5AB19412
 P 4300 4050
-F 0 "C12" H 4325 4150 50  0000 L CNN
+F 0 "C13" H 4325 4150 50  0000 L CNN
 F 1 "100uF" H 4325 3950 50  0000 L CNN
 F 2 "m2_simcom_7100:CP_Tantalum_Case-B_EIA-3528-21_Reflow" H 4300 4050 50  0001 C CNN
@@
 $EndComp
 $Comp
-L C C13
+L C C14
 U 1 1 5AB19443
 P 4500 4050
-F 0 "C13" H 4525 4150 50  0000 L CNN
+F 0 "C14" H 4525 4150 50  0000 L CNN
 F 1 "1uF" H 4525 3950 50  0000 L CNN
 F 2 "Capacitors_SMD:C_0603" H 4538 3900 50  0001 C CNN
@@
 $EndComp
 $Comp
-L CP1 C15
+L CP1 C16
 U 1 1 5AB194A7
 P 7300 4050
-F 0 "C15" H 7325 4150 50  0000 L CNN
+F 0 "C16" H 7325 4150 50  0000 L CNN
 F 1 "100uF" H 7325 3950 50  0000 L CNN
 F 2 "m2_simcom_7100:CP_Tantalum_Case-B_EIA-3528-21_Reflow" H 7300 4050 50  0001 C CNN
@@
 $EndComp
 $Comp
-L R R10
+L R R11
 U 1 1 5AB195E5
 P 6950 4100
-F 0 "R10" H 7100 4150 50  0000 C CNN
+F 0 "R11" H 7100 4150 50  0000 C CNN
 F 1 "180k" H 7100 4050 50  0000 C CNN
 F 2 "Resistors_SMD:R_0603" V 6880 4100 50  0001 C CNN
@@
 $EndComp
 $Comp
-L R R11
+L R R12
 U 1 1 5AB19636
 P 6950 4700
-F 0 "R11" H 7100 4750 50  0000 C CNN
+F 0 "R12" H 7100 4750 50  0000 C CNN
 F 1 "47k" H 7100 4650 50  0000 C CNN
 F 2 "Resistors_SMD:R_0603" V 6880 4700 50  0001 C CNN
@@
 $EndComp
 $Comp
-L GND #PWR022
+L GND #PWR026
 U 1 1 5AB19681
 P 6950 4900
-F 0 "#PWR022" H 6950 4650 50  0001 C CNN
+F 0 "#PWR026" H 6950 4650 50  0001 C CNN
 F 1 "GND" H 6950 4750 50  0000 C CNN
 F 2 "" H 6950 4900 50  0001 C CNN
@@
 $EndComp
 $Comp
-L GND #PWR023
+L GND #PWR027
 U 1 1 5AB198DF
 P 7300 4250
-F 0 "#PWR023" H 7300 4000 50  0001 C CNN
+F 0 "#PWR027" H 7300 4000 50  0001 C CNN
 F 1 "GND" H 7300 4100 50  0000 C CNN
 F 2 "" H 7300 4250 50  0001 C CNN
@@
 $EndComp
 $Comp
-L GND #PWR024
+L GND #PWR028
 U 1 1 5AB1991A
 P 7600 4250
-F 0 "#PWR024" H 7600 4000 50  0001 C CNN
+F 0 "#PWR028" H 7600 4000 50  0001 C CNN
 F 1 "GND" H 7600 4100 50  0000 C CNN
 F 2 "" H 7600 4250 50  0001 C CNN
@@
 $EndComp
 $Comp
-L GND #PWR025
+L GND #PWR029
 U 1 1 5AB19B43
 P 4300 4250
-F 0 "#PWR025" H 4300 4000 50  0001 C CNN
+F 0 "#PWR029" H 4300 4000 50  0001 C CNN
 F 1 "GND" H 4300 4100 50  0000 C CNN
 F 2 "" H 4300 4250 50  0001 C CNN
@@
 $EndComp
 $Comp
-L GND #PWR026
+L GND #PWR030
 U 1 1 5AB19B9E
 P 4500 4250
-F 0 "#PWR026" H 4500 4000 50  0001 C CNN
+F 0 "#PWR030" H 4500 4000 50  0001 C CNN
 F 1 "GND" H 4500 4100 50  0000 C CNN
 F 2 "" H 4500 4250 50  0001 C CNN
@@
 Connection ~ 4300 3850
 $Comp
-L C C16
+L C C17
 U 1 1 5AB19573
 P 7600 4050
-F 0 "C16" H 7625 4150 50  0000 L CNN
+F 0 "C17" H 7625 4150 50  0000 L CNN
 F 1 "100nF" H 7625 3950 50  0000 L CNN
 F 2 "Capacitors_SMD:C_0603" H 7638 3900 50  0001 C CNN
@@
 $EndBitmap
 $Comp
-L RT9059 U2
+L RT9059 U3
 U 1 1 5AB559CB
 P 5950 4150
-F 0 "U2" H 5700 4600 60  0000 C CNN
+F 0 "U3" H 5700 4600 60  0000 C CNN
 F 1 "RT9059" H 6100 4600 60  0000 C CNN
 F 2 "m2_simcom_7100:DFN-10-1EP_3x3mm_Pitch0.5mm" H 5850 4350 60  0001 C CNN
@@
 Connection ~ 6500 3950
 $Comp
-L R R9
+L R R10
 U 1 1 5AB56208
 P 6600 4050
-F 0 "R9" H 6750 4100 50  0000 C CNN
+F 0 "R10" H 6750 4100 50  0000 C CNN
 F 1 "100k" H 6750 4000 50  0000 C CNN
 F 2 "Resistors_SMD:R_0603" V 6530 4050 50  0001 C CNN
@@
 $EndComp
 $Comp
-L C C14
+L C C15
 U 1 1 5AB57BE3
 P 4750 4450
-F 0 "C14" H 4775 4550 50  0000 L CNN
+F 0 "C15" H 4775 4550 50  0000 L CNN
 F 1 "1uF" H 4775 4350 50  0000 L CNN
 F 2 "Capacitors_SMD:C_0603" H 4788 4300 50  0001 C CNN
@@
 Connection ~ 4750 4250
 $Comp
-L GND #PWR027
+L GND #PWR031
 U 1 1 5AB58392
 P 4750 4650
-F 0 "#PWR027" H 4750 4400 50  0001 C CNN
+F 0 "#PWR031" H 4750 4400 50  0001 C CNN
 F 1 "GND" H 4750 4500 50  0000 C CNN
 F 2 "" H 4750 4650 50  0001 C CNN
